File: sendai/sendai.brd (EAGLE design)
At the start: 43 x 43 mm, 4 parts

Commit message: lead switch
Parts:
- U$4: value RESISTOR -> LEAD_SWITCH; device RESISTOR:RESISTOR -> LEAD_SWITCH:LEAD_SWITCH
Connections:
- net N$1: now also U$4.P$3; no longer U$4.1
- net N$3: now also U$4.P$4; no longer U$4.2
Routing:
- net N$1: track 33.8 -> 35.2 mm
- net N$3: track 5.23 -> 6.15 mm
Changed lines of the file:
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@@
 <element name="U$2" library="CONNECTER" package="CON2" value="CON2" x="13.335" y="9.525" rot="R330"/>
 <element name="U$3" library="CONNECTER" package="CON2" value="CON2" x="29.845" y="9.525" rot="R210"/>
-<element name="U$4" library="RESISTOR" package="RESISTOR" value="RESISTOR" x="6.985" y="20.955" rot="R90"/>
+<element name="U$4" library="LEAD_SWITCH" package="LEAD_SWITCH" value="LEAD_SWITCH" x="6.985" y="20.955" rot="R90"/>
 </elements>
 <signals>
@@
 <wire x1="29.21" y1="5.715" x2="30.743025" y2="6.613025" width="1.016" layer="1"/>
 <wire x1="30.94485" y1="10.16" x2="30.743025" y2="6.613025" width="1.016" layer="1"/>
-<contactref element="U$4" pad="1"/>
-<wire x1="6.985" y1="15.875" x2="7.356971875" y2="14.868028125" width="1.016" layer="1"/>
-<wire x1="7.356971875" y1="14.868028125" x2="12.235146875" y2="10.16" width="1.016" layer="1"/>
+<contactref element="U$4" pad="P$3"/>
+<wire x1="6.985" y1="14.955" x2="6.985" y2="11.43" width="1.016" layer="1"/>
+<wire x1="6.985" y1="11.43" x2="8.255" y2="10.16" width="1.016" layer="1"/>
+<wire x1="8.255" y1="10.16" x2="12.235146875" y2="10.16" width="1.016" layer="1"/>
 </signal>
 <signal name="N$2">
@@
 <signal name="N$3">
 <contactref element="U$1" pad="+1"/>
-<contactref element="U$4" pad="2"/>
-<wire x1="7.34" y1="20.955" x2="7.34" y2="25.68" width="1.016" layer="1"/>
-<wire x1="7.34" y1="25.68" x2="6.985" y2="26.035" width="1.016" layer="1"/>
+<contactref element="U$4" pad="P$4"/>
+<wire x1="6.985" y1="26.955" x2="6.985" y2="21.31" width="1.016" layer="1"/>
+<wire x1="6.985" y1="21.31" x2="7.34" y2="20.955" width="1.016" layer="1"/>
 </signal>
 </signals>
