File: sendai/sendai.sch (EAGLE design)
At the start: 4 parts

Commit message: lead switch
Parts:
- U$4: value RESISTOR -> LEAD_SWITCH; device RESISTOR:RESISTOR -> LEAD_SWITCH:LEAD_SWITCH
Connections:
- net N$1: now also U$4.P$1; no longer U$4.1
- net N$3: now also U$4.P$2; no longer U$4.2
Changed lines of the file:
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@@
 <part name="U$2" library="CONNECTER" deviceset="CON2" device=""/>
 <part name="U$3" library="CONNECTER" deviceset="CON2" device=""/>
-<part name="U$4" library="RESISTOR" deviceset="RESISTOR" device=""/>
+<part name="U$4" library="LEAD_SWITCH" deviceset="LEAD_SWITCH" device=""/>
 </parts>
 <sheets>
@@
 <instance part="U$2" gate="G$1" x="45.72" y="40.64" rot="R270"/>
 <instance part="U$3" gate="G$1" x="71.12" y="40.64" rot="R270"/>
-<instance part="U$4" gate="G$1" x="35.56" y="66.04" rot="R180"/>
+<instance part="U$4" gate="G$1" x="35.56" y="66.04"/>
 </instances>
 <busses>
@@
 <pinref part="U$2" gate="G$1" pin="P$1"/>
 <wire x1="45.72" y1="43.18" x2="45.72" y2="53.34" width="0.1524" layer="91"/>
-<pinref part="U$4" gate="G$1" pin="1"/>
 <wire x1="45.72" y1="66.04" x2="45.72" y2="53.34" width="0.1524" layer="91"/>
 <junction x="45.72" y="53.34"/>
+<pinref part="U$4" gate="G$1" pin="P$1"/>
+<wire x1="43.18" y1="66.04" x2="45.72" y2="66.04" width="0.1524" layer="91"/>
 </segment>
 </net>
@@
 <segment>
 <pinref part="U$1" gate="G$1" pin="+"/>
-<pinref part="U$4" gate="G$1" pin="2"/>
 <wire x1="25.4" y1="48.26" x2="25.4" y2="66.04" width="0.1524" layer="91"/>
+<pinref part="U$4" gate="G$1" pin="P$2"/>
+<wire x1="27.94" y1="66.04" x2="25.4" y2="66.04" width="0.1524" layer="91"/>
 </segment>
 </net>
